File: FPS 100/Backplane/Backplane.kicad_sch (KiCad schematic)
At the start: 28 parts

Commit message: 2026/1/4
Parts:
- added UNIBUS_XFER_J1: Conn_02x25_Odd_Even, symbol Connector_Generic:Conn_02x25_Odd_Even
Connections:
- net !A1CLK: now also 4408_P3_J1.15
- net !A2CLK: now also 4408_P3_J1.14
- net !CBCLK1: now also 4408_P3_J1.8
- net !CBCLK2: now also 4408_P3_J1.7
- net !DPLCLK: now also 4408_P3_J1.16
- net !DPRCLK: now also 4408_P3_J1.17
- net !FACLK: now also 4408_P3_J1.19
- net !FMCLK: now also 4408_P3_J1.13
- net !MCLK: now also 4408_P3_J1.21
- net !SPCLK: now also 4408_P3_J1.5
- net !T75: now also 4408_P3_J1.11
- net !TMCLK: now also 4408_P3_J1.10
- net !WRT*: now also 4408_P3_J1.6
- net !WRTL*: now also 4408_P3_J1.18
- net 376IN*: now also 4408_P3_J2.57
- net 376LD*: now also 4408_P3_J2.58
- net 377IN*: now also 4408_P3_J1.39
- net 377LD*: now also 4408_P3_J1.37
- net ABORT*: now also 4408_P3_J1.50
- net BS2A1: now also 4408_P3_J2.12
- net BS2A2: now also 4408_P3_J2.18
- net CB14*: now also 4408_P3_J2.47
- net CB15*: now also 4408_P3_J2.48
- net CB16*: now also 4408_P3_J2.49
- net CB17*: now also 4408_P3_J2.50
- net CB18*: now also 4408_P3_J2.51
- net CB19*: now also 4408_P3_J2.52
- net CB2A1E*: now also 4408_P3_J2.56
- net CB2A2E*: now also 4408_P3_J2.20
- net CB2A2M*: now also 4408_P3_J2.19
- net CBCLKE*: now also 4408_P3_J1.97
- net DA08*: now also 4421_PDP_IF_J1.12
- net DA09*: now also 4421_PDP_IF_J1.14
- net DA10*: now also 4421_PDP_IF_J1.16
- net DA11*: now also 4421_PDP_IF_J1.18
- net DA12*: now also 4421_PDP_IF_J1.24
- net DA13*: now also 4421_PDP_IF_J1.26
- net DA14*: now also 4421_PDP_IF_J1.28
- net DA15*: now also 4421_PDP_IF_J1.30
- net DA2PNL: now also 4408_P3_J1.83
- net DALD*: now also 4408_P3_J1.105
- net DBLSW*: now also 4408_P3_J1.23
- net DCHO01*: now also 4421_PDP_IF_J1.59
- net DMA00*: now also 4421_PDP_IF_J1.62
- net DMA02*: now also 4421_PDP_IF_J1.66
- net DMA03*: now also 4421_PDP_IF_J1.68
- net DMA04*: now also 4421_PDP_IF_J2.10
- net DMA05*: now also 4421_PDP_IF_J2.12
- net DMA06*: now also 4421_PDP_IF_J2.14
- net DMA07*: now also 4421_PDP_IF_J2.16
- net DMA08*: now also 4421_PDP_IF_J2.39
- net DMA09*: now also 4421_PDP_IF_J2.41
- net DMA10*: now also 4421_PDP_IF_J2.43
- net DMA11*: now also 4421_PDP_IF_J2.45
- net DMA12*: now also 4421_PDP_IF_J2.79
- net DMA13*: now also 4421_PDP_IF_J2.81
- net DMA14*: now also 4421_PDP_IF_J2.83
- net DMA15*: now also 4421_PDP_IF_J2.85
- net DP2A1: now also 4408_P3_J2.5
- net DP2A2E: now also 4408_P3_J1.115
- net DP2A2M: now also 4408_P3_J2.6
- net DPA2PNL*: now also 4408_P3_J2.54
- net DPEBS02*: now also 4408_P3_J1.61, 4429_FMT_J1.17
- net DPEBS03*: now also 4408_P3_J1.63, 4429_FMT_J1.19
- net DPEBS04*: now also 4408_P3_J1.65, 4429_FMT_J1.31
- net DPEBS05*: now also 4408_P3_J1.67, 4429_FMT_J1.33
- net DPEBS06*: now also 4408_P3_J1.69, 4429_FMT_J1.35
- net DPEBS07*: now also 4408_P3_J1.71, 4429_FMT_J1.37
- net DPEBS08*: now also 4408_P3_J1.102, 4429_FMT_J1.57
- net DPEBS09*: now also 4408_P3_J1.104, 4429_FMT_J1.59
- net DPEBS10*: now also 4408_P3_J1.106, 4429_FMT_J1.61
- net DPEBS11*: now also 4408_P3_J1.108, 4429_FMT_J1.63
- net DPMBS00*: now also 4408_P3_J2.25, 4429_FMT_J1.71
- net DPMBS01*: now also 4408_P3_J2.26, 4429_FMT_J1.73
- net DPMBS02*: now also 4408_P3_J2.27, 4429_FMT_J1.75
- net DPMBS03*: now also 4408_P3_J2.28, 4429_FMT_J1.77
- net DPMBS04*: now also 4408_P3_J2.67, 4429_FMT_J1.87
- net DPMBS05*: now also 4408_P3_J2.68, 4429_FMT_J1.89
- net DPMBS06*: now also 4408_P3_J2.69, 4429_FMT_J1.91
- net DPMBS07*: now also 4408_P3_J2.70, 4429_FMT_J1.93
- net DPMBS08*: now also 4408_P3_J2.71, 4429_FMT_J2.15
- net DPMBS09*: now also 4408_P3_J2.72, 4429_FMT_J2.17
- net DPMBS10*: now also 4408_P3_J2.73, 4421_PDP_IF_J1.65, 4429_FMT_J2.19
- net DPMBS11*: now also 4408_P3_J2.74, 4421_PDP_IF_J2.51, 4429_FMT_J2.21
- net DPMBS12*: now also 4408_P3_J2.87, 4421_PDP_IF_J1.51, 4429_FMT_J2.35
- net DPMBS13*: now also 4408_P3_J2.88, 4421_PDP_IF_J1.53, 4429_FMT_J2.37
- net DPMBS14*: now also 4408_P3_J2.89, 4421_PDP_IF_J1.55, 4429_FMT_J2.39
- net DPMBS15*: now also 4408_P3_J2.90, 4421_PDP_IF_J1.57, 4429_FMT_J2.41
- net DPMBS16*: now also 4408_P3_J2.91, 4421_PDP_IF_J1.81, 4429_FMT_J2.51
- net DPMBS17*: now also 4408_P3_J2.92, 4421_PDP_IF_J1.83, 4429_FMT_J2.53
- net DPMBS18*: now also 4408_P3_J2.93, 4421_PDP_IF_J1.85, 4429_FMT_J2.55
- net DPMBS19*: now also 4408_P3_J2.94, 4421_PDP_IF_J1.87, 4429_FMT_J2.57
- net DPMBS20*: now also 4408_P3_J2.101, 4421_PDP_IF_J1.89, 4429_FMT_J2.69
- net DPMBS21*: now also 4408_P3_J2.102, 4421_PDP_IF_J1.91, 4429_FMT_J2.71
- net DPMBS22*: now also 4408_P3_J2.103, 4421_PDP_IF_J2.67, 4429_FMT_J2.73
- net DPMBS23*: now also 4408_P3_J2.104, 4421_PDP_IF_J2.69, 4429_FMT_J2.75
- net DPMBS24*: now also 4408_P3_J2.109, 4421_PDP_IF_J2.71, 4429_FMT_J2.89
- net DPMBS25*: now also 4408_P3_J2.110, 4421_PDP_IF_J2.73, 4429_FMT_J2.91
- net DPMBS26*: now also 4408_P3_J2.111, 4421_PDP_IF_J2.75, 4429_FMT_J2.93
- net DPMBS27*: now also 4408_P3_J2.112, 4421_PDP_IF_J2.77, 4429_FMT_J2.95
- net EX2PNL*: now also 4408_P3_J1.86
- net FADD*: now also 4408_P3_J2.86
- net FLAG0: now also 4408_P3_J1.57
- net FLAG1: now also 4408_P3_J1.58
- net FLAG2: now also 4408_P3_J1.59
- net FLAG3: now also 4408_P3_J1.60
- net FMUL*: now also 4408_P3_J1.22
- net HD2DP: now also 4408_P3_J1.33
- net IN100: now also 4408_P3_J2.40, 4421_PDP_IF_J1.38
- net INT2A1E*: now also 4408_P3_J2.37
- net INTR*: now also 4421_PDP_IF_J1.39
- net INTR1*: now also 4408_P3_J1.95
- net INTU*: now also 4408_P3_J1.43
- net IODRDY*: now also 4421_PDP_IF_J1.10
- net IODRDYQ: now also 4408_P3_J1.103
- net LDOMA*: now also 4408_P3_J1.88
- net MA2PNL: now also 4408_P3_J1.94
- net MA=SUP*: now also 4408_P3_J1.45
- net MD02*: now also 4429_FMT_J1.18
- net MD03*: now also 4429_FMT_J1.20
- net MD04*: now also 4429_FMT_J1.32
- net MD05*: now also 4429_FMT_J1.34
- net MD06*: now also 4429_FMT_J1.36
- net MD07*: now also 4429_FMT_J1.38
- net MD08*: now also 4429_FMT_J1.58
- net MD09*: now also 4429_FMT_J1.60
- net MD10*: now also 4429_FMT_J1.62
- net MD11*: now also 4429_FMT_J1.64
- net MD12*: now also 4429_FMT_J1.72
- net MD13*: now also 4429_FMT_J1.74
- net MD14*: now also 4429_FMT_J1.76
- net MD15*: now also 4429_FMT_J1.78
- net MD16*: now also 4429_FMT_J1.88
- net MD17*: now also 4429_FMT_J1.90
- net MD18*: now also 4429_FMT_J1.92
- net MD19*: now also 4429_FMT_J1.94
- net MD20*: now also 4429_FMT_J2.16
- net MD21*: now also 4429_FMT_J2.18
- net MD22*: now also 4429_FMT_J2.20
- net MD23*: now also 4429_FMT_J2.22
- net MD24*: now also 4429_FMT_J2.36
- net MD25*: now also 4429_FMT_J2.38
- net MD26*: now also 4429_FMT_J2.40
- net MD27*: now also 4429_FMT_J2.42
- net MD28*: now also 4429_FMT_J2.52
- net MD29*: now also 4429_FMT_J2.54
- net MD2A2: now also 4408_P3_J2.11
- net MD30*: now also 4429_FMT_J2.56
- net MD31*: now also 4429_FMT_J2.58
- net MD32*: now also 4429_FMT_J2.70
- net MD33*: now also 4429_FMT_J2.72
- net MD34*: now also 4429_FMT_J2.74
- net MD35*: now also 4429_FMT_J2.76
- net MD36*: now also 4429_FMT_J2.90
- net MD37*: now also 4429_FMT_J2.92
- net MD38*: now also 4429_FMT_J2.94
- net MD39*: now also 4429_FMT_J2.96
- net MD3BSY: now also 4408_P3_J1.74
- net MD3REJ: now also 4408_P3_J1.90
- net MDCA1: now also 4421_PDP_IF_J1.35
- net MDCR1Q*: now also 4421_PDP_IF_J1.60
- net MDCR3*: now also 4408_P3_J1.89
- net MDI02: now also 4429_FMT_J1.23
- net MDI03: now also 4429_FMT_J1.24
- net MDI04: now also 4429_FMT_J1.25
- net MDI05: now also 4429_FMT_J1.26
- net MDI06: now also 4429_FMT_J1.39
- net MDI07: now also 4429_FMT_J1.40
- net MDI08: now also 4429_FMT_J1.41
- net MDI09: now also 4429_FMT_J1.42
- net MDI10: now also 4429_FMT_J1.43
- net MDI11: now also 4429_FMT_J1.44
- net MDI12: now also 4429_FMT_J1.81
- net MDI13: now also 4429_FMT_J1.82
- net MDI14: now also 4429_FMT_J1.83
- net MDI15: now also 4429_FMT_J1.84
- net MDI16: now also 4429_FMT_J1.85
- net MDI17: now also 4429_FMT_J1.86
- net MDI18: now also 4429_FMT_J2.11
- net MDI19: now also 4429_FMT_J2.12
- net MDI20: now also 4429_FMT_J2.13
- net MDI21: now also 4429_FMT_J2.14
- net MDI22: now also 4429_FMT_J2.29
- net MDI23: now also 4429_FMT_J2.30
- net MDI24: now also 4429_FMT_J2.31
- net MDI25: now also 4429_FMT_J2.32
- net MDI26: now also 4429_FMT_J2.33
- net MDI27: now also 4429_FMT_J2.34
- net MDI28: now also 4429_FMT_J2.63
- net MDI29: now also 4429_FMT_J2.64
- net MDI30: now also 4429_FMT_J2.65
- net MDI31: now also 4429_FMT_J2.66
- net MDI32: now also 4429_FMT_J2.67
- net MDI33: now also 4429_FMT_J2.68
- net MDI34: now also 4429_FMT_J2.83
- net MDI35: now also 4429_FMT_J2.84
- net MDI36: now also 4429_FMT_J2.85
- net MDI37: now also 4429_FMT_J2.86
- net MDI38: now also 4429_FMT_J2.87
- net MDI39: now also 4429_FMT_J2.88
- net MDUSE*: now also 4408_P3_J1.96
- net MDWRT*: now also 4421_PDP_IF_J1.37
- net OUT*: now also 4408_P3_J1.55, 4421_PDP_IF_J1.43
- net PAUSE1*: now also 4408_P3_J1.100
- net PNL00*: now also 4408_P3_J1.24
- net PNL01*: now also 4408_P3_J1.26
- net PNL02*: now also 4408_P3_J1.28
- net PNL03*: now also 4408_P3_J1.30
- net PNL04*: now also 4408_P3_J1.32
- net PNL05*: now also 4408_P3_J1.34
- net PNL06*: now also 4408_P3_J1.36
- net PNL07*: now also 4408_P3_J1.38
- net PNL08*: now also 4408_P3_J1.40, 4421_PDP_IF_J1.11
- net PNL09*: now also 4408_P3_J1.42, 4421_PDP_IF_J1.13
- net PNL10*: now also 4408_P3_J1.44, 4421_PDP_IF_J1.15
- net PNL11*: now also 4408_P3_J1.46, 4421_PDP_IF_J1.17
- net PNL12*: now also 4408_P3_J1.62, 4421_PDP_IF_J1.23
- net PNL13*: now also 4408_P3_J1.64, 4421_PDP_IF_J1.25
- net PNL14*: now also 4408_P3_J1.66, 4421_PDP_IF_J1.27
- net PNL15*: now also 4408_P3_J1.68, 4421_PDP_IF_J1.29
- net PNL2DP: now also 4408_P3_J1.72
- net PNL2MA*: now also 4408_P3_J2.38
- net PNL2MD*: now also 4408_P3_J1.54
- net PNL2PSA*: now also 4408_P3_J1.91
- net PNL2TMA*: now also 4408_P3_J2.39
- net PS03*: now also 4408_P3_J2.60
- net PS06*: now also 4408_P3_J2.59
- net PS07*B: now also 4408_P3_J2.8
- net PS08*: now also 4408_P3_J2.61
- net PS09*: now also 4408_P3_J2.62
- net PS0WRT: now also 4408_P3_J2.21
- net PS10*: now also 4408_P3_J2.63
- net PS11*: now also 4408_P3_J2.64
- net PS12*: now also 4408_P3_J2.65
- net PS13*: now also 4408_P3_J2.66
- net PS14*: now also 4408_P3_J2.81
- net PS15*: now also 4408_P3_J2.82
- net PS16*: now also 4408_P3_J2.83
- net PS17*: now also 4408_P3_J2.84
- net PS18*: now also 4408_P3_J2.85
- net PS19*: now also 4408_P3_J2.105
- net PS1WRT: now also 4408_P3_J2.22
- net PS20*: now also 4408_P3_J2.106
- net PS21*: now also 4408_P3_J2.107
- net PS22*: now also 4408_P3_J2.108
- net PS2WRT: now also 4408_P3_J2.23
- net PS33*: now also 4408_P3_J2.13
- net PS35*: now also 4408_P3_J2.14
- net PS36*: now also 4408_P3_J2.15
- net PS37*: now also 4408_P3_J2.16
- net PS38*: now also 4408_P3_J2.17
- net PS3WRT: now also 4408_P3_J2.24
- net PS56*: now also 4408_P3_J2.95
- net PS57*: now also 4408_P3_J2.96
- net PS59*: now also 4408_P3_J2.97
- net PS61*: now also 4408_P3_J2.98
- net PS63*: now also 4408_P3_J2.99
- net PSA2PNL: now also 4408_P3_J1.92
- net PSACLKE*: now also 4408_P3_J1.98
- net PSH2DP: now also 4408_P3_J1.112
- net PSL2DP: now also 4408_P3_J1.111
- net PSZIP*: now also 4408_P3_J1.49
- net PUSHA1: now also 4408_P3_J2.35
- net PUSHA2: now also 4408_P3_J2.36
- net RDOMA*: now also 4408_P3_J1.87
- net REFSYNC*: now also 4408_P3_J2.53
- net RTM*: now also 4408_P3_J2.55
- net RUN*: now also 4408_P3_J1.47, 4421_PDP_IF_J1.93
- net SETATMA*: now also 4408_P3_J1.85
- net SP2ADDR: now also 4408_P3_J1.110
- net SPA2PNL: now also 4408_P3_J1.82
- net SPD2PNL: now also 4408_P3_J1.81
- net SPEC*: now also 4408_P3_J2.10
- net SPIN*: now also 4408_P3_J1.51
- net STA2PNL: now also 4408_P3_J1.84
- net TM2A1: now also 4408_P3_J2.34
- net TM2PNL: now also 4408_P3_J1.48
- net TMA2PNL: now also 4408_P3_J1.93
- net TSPIN: now also 4408_P3_J1.52
- net USECB*: now also 4408_P3_J2.7
- net USEPNL*: now also 4408_P3_J1.56
- net USEPSA*: now also 4408_P3_J1.53
- net WRTEXP: now also 4408_P3_J1.109
- net WRTHM: now also 4408_P3_J1.113
- net WRTLM: now also 4408_P3_J1.114
- net Y2A1: now also 4408_P3_J2.33
- net Y2A2: now also 4408_P3_J2.9
- net I+H10: now reaches 4429_FMT_J1.10
- net I+H10: now also 4421_PDP_IF_J2.46
- net I+H13: now reaches 4429_FMT_J1.11
- net I+H13: now also 4421_PDP_IF_J2.80
- net I+H14: now reaches 4429_FMT_J1.12
- net I+H14: now also 4421_PDP_IF_J2.82
- net CTCLK: now reaches 4429_FMT_J1.13
- net B2MDI: now reaches 4429_FMT_J1.14
- net B2MDI: now also 4421_PDP_IF_J1.41
- net B2IO: now reaches 4429_FMT_J1.15
- net BH2HD: now reaches 4429_FMT_J1.16
- net BH2HD: now also 4421_PDP_IF_J2.96
- net HD00A: now reaches 4429_FMT_J1.27
- net HD01A: now reaches 4429_FMT_J1.29
- net HD02A: now reaches 4429_FMT_J1.30
- net B0CLK: now reaches 4429_FMT_J1.48
- net B0CLK: now also 4421_PDP_IF_J1.36, 4429_FMT_J1.5
- net HD03A: now reaches 4429_FMT_J1.51
- net HD04B: now reaches 4429_FMT_J1.52
- net HD05B: now reaches 4429_FMT_J1.53
- net HD06B: now reaches 4429_FMT_J1.54
- net HD07B: now reaches 4429_FMT_J1.55
- net HD08B: now reaches 4429_FMT_J1.56
- net BUF2CLK: now reaches 4429_FMT_J1.6
- net BUF2CLK: now also 4421_PDP_IF_J1.48
- net OVFL*: now reaches 4429_FMT_J1.66
- net OVFL*: now also 4421_PDP_IF_J1.70
- net HD04A: now reaches 4429_FMT_J1.67
- net HD05A: now reaches 4429_FMT_J1.68
- net HD06A: now reaches 4429_FMT_J1.69
- net RPDP: now reaches 4429_FMT_J1.7
- net HD07A: now reaches 4429_FMT_J1.70
- net BL2HD: now reaches 4429_FMT_J1.79
- net BL2HD: now also 4421_PDP_IF_J2.94
- net UNFL*: now reaches 4429_FMT_J1.80
- net UNFL*: now also 4421_PDP_IF_J1.72
- net I+H09: now reaches 4429_FMT_J1.9
- net I+H09: now also 4421_PDP_IF_J2.44
- net PNL2DBL*: now reaches 4408_P3_J1.101
- net IOACK*: now reaches 4408_P3_J1.107
- net IOACK*: now also 4421_PDP_IF_J1.46
- net NCP*: now reaches 4408_P3_J1.116
- net !M1CLK: now reaches 4408_P3_J1.12
- net !IOCLK: now reaches 4408_P3_J1.20
- net IHRSET*: now reaches 4408_P3_J1.25
- net LDSR*: now reaches 4408_P3_J1.27
- net LDSR*: now also 4421_PDP_IF_J2.74, 4421_PDP_IF_J2.86
- net PHALT*: now reaches 4408_P3_J1.29
- net TRIGQ*: now reaches 4408_P3_J1.31
- net INTIND: now reaches 4408_P3_J1.35
- net INTA: now reaches 4408_P3_J1.41
- net SR2HD*: now reaches 4408_P3_J1.70
- net SR2HD*: now also 4421_PDP_IF_J2.92
- net SNSB: now reaches 4408_P3_J1.73
- net IN: now reaches 4408_P3_J1.75
- net SNSA: now reaches 4408_P3_J1.76
- net INTEN: now reaches 4408_P3_J1.77
- net INTEN: now also 4421_PDP_IF_J1.40
- net IONTA: now reaches 4408_P3_J1.78
- net DP2IO*: now reaches 4408_P3_J1.79
- net IORST*: now reaches 4408_P3_J1.80
- net !WRTR: now reaches 4408_P3_J1.9
- net LDFN*: now reaches 4408_P3_J1.99
- net LDFN*: now also 4421_PDP_IF_J2.72, 4421_PDP_IF_J2.84
- net EXTNT: now reaches 4408_P3_J2.100
- net INTCP: now reaches 4408_P3_J2.113
- net LT2HD*: now reaches 4408_P3_J2.114
- net LT2HD*: now also 4421_PDP_IF_J2.88
- net EXTCLK{408}: now reaches 4408_P3_J2.115
- net FN2HD*: now reaches 4408_P3_J2.116
- net FN2HD*: now also 4421_PDP_IF_J2.90
- net HD00: now reaches 4408_P3_J2.29
- net HD00: now also 4421_PDP_IF_J1.74, 4429_FMT_J2.25
- net HD01: now reaches 4408_P3_J2.30
- net HD01: now also 4421_PDP_IF_J1.76, 4429_FMT_J2.26
- net HD02: now reaches 4408_P3_J2.31
- net HD02: now also 4421_PDP_IF_J1.78, 4429_FMT_J2.27
- net HD03: now reaches 4408_P3_J2.32
- net HD03: now also 4421_PDP_IF_J1.80, 4429_FMT_J2.28
- net HD04: now reaches 4408_P3_J2.41
- net HD04: now also 4421_PDP_IF_J2.24, 4429_FMT_J2.43
- net HD05: now reaches 4408_P3_J2.42
- net HD05: now also 4421_PDP_IF_J2.26, 4429_FMT_J2.44
- net HD06: now reaches 4408_P3_J2.43
- net HD06: now also 4421_PDP_IF_J2.28, 4429_FMT_J2.45
- net HD07: now reaches 4408_P3_J2.44
- net HD07: now also 4421_PDP_IF_J2.30, 4429_FMT_J2.46
- net HD08: now reaches 4408_P3_J2.45
- net HD08: now also 4421_PDP_IF_J2.36, 4429_FMT_J2.47
- net HD09: now reaches 4408_P3_J2.46
- net HD09: now also 4421_PDP_IF_J2.38, 4429_FMT_J2.48
- net HD10: now reaches 4408_P3_J2.75
- net HD10: now also 4421_PDP_IF_J2.40, 4429_FMT_J2.77
- net HD11: now reaches 4408_P3_J2.76
- net HD11: now also 4421_PDP_IF_J2.42, 4429_FMT_J2.78
- net HD12: now reaches 4408_P3_J2.77
- net HD12: now also 4421_PDP_IF_J2.58, 4429_FMT_J2.79
- net HD13: now reaches 4408_P3_J2.78
- net HD13: now also 4421_PDP_IF_J2.60, 4429_FMT_J2.80
- net HD14: now reaches 4408_P3_J2.79
- net HD14: now also 4421_PDP_IF_J2.62, 4429_FMT_J2.81
- net HD15: now reaches 4408_P3_J2.80
- net HD15: now also 4421_PDP_IF_J2.64, 4429_FMT_J2.82
- net HD13A: now reaches 4429_FMT_J2.10
- net HD14A: now reaches 4429_FMT_J2.23
- net HD15A: now reaches 4429_FMT_J2.24
- net HD08A: now reaches 4429_FMT_J2.5
- net B2CLK: now reaches 4429_FMT_J2.59
- net B2CLK: now also 4421_PDP_IF_J1.45, 4429_FMT_J2.62
- net HD09A: now reaches 4429_FMT_J2.6
- net HD10A: now reaches 4429_FMT_J2.7
- net HD11A: now reaches 4429_FMT_J2.8
- net HD12A: now reaches 4429_FMT_J2.9
- net B2ID: now reaches 4421_PDP_IF_J1.42
- net INTPIN: now reaches 4421_PDP_IF_J1.44
- net BUSA17*: now reaches 4421_PDP_IF_J1.47
- net BUSA17*: now also UNIBUS_XFER_J1.35 (Pin_35)
- net HINTIND: now reaches 4421_PDP_IF_J1.49
- net CTLCLK: now reaches 4421_PDP_IF_J1.50
- net BUSA16*: now reaches 4421_PDP_IF_J1.61
- net BUSA16*: now also UNIBUS_XFER_J1.33 (Pin_33)
- net BUSA15*: now reaches 4421_PDP_IF_J1.63
- net BUSA15*: now also UNIBUS_XFER_J1.31 (Pin_31)
- net DAM01*: now reaches 4421_PDP_IF_J1.64
- net BUSA14*: now reaches 4421_PDP_IF_J1.67
- net BUSA14*: now also UNIBUS_XFER_J1.29 (Pin_29)
- net BUSA13*: now reaches 4421_PDP_IF_J1.69
- net BUSA13*: now also UNIBUS_XFER_J1.27 (Pin_27)
- net BUSD15*: now reaches 4421_PDP_IF_J1.71
- net BUSD15*: now also UNIBUS_XFER_J1.32 (Pin_32)
- net BUSD14*: now reaches 4421_PDP_IF_J1.73
- net BUSD14*: now also UNIBUS_XFER_J1.30 (Pin_30)
- net BUSD13*: now reaches 4421_PDP_IF_J1.77
- net BUSD13*: now also UNIBUS_XFER_J1.28 (Pin_28)
- net BUSD12*: now reaches 4421_PDP_IF_J1.79
- net BUSD12*: now also UNIBUS_XFER_J1.26 (Pin_26)
- net INTPOUT: now reaches 4421_PDP_IF_J1.92
- net BUSNPGIN: now reaches 4421_PDP_IF_J1.94
- net BUSNPGIN: now also UNIBUS_XFER_J1.47 (Pin_47)
- net BUSBGIN: now reaches 4421_PDP_IF_J1.95
- net BUSBGIN: now also UNIBUS_XFER_J1.49 (Pin_49)
- net BUSBBSY*: now reaches 4421_PDP_IF_J1.96
- net BUSBBSY*: now also UNIBUS_XFER_J1.45 (Pin_45)
- net BUSA11*: now reaches 4421_PDP_IF_J2.11
- net BUSA11*: now also UNIBUS_XFER_J1.23 (Pin_23)
- net HADRCLK*: now reaches 4421_PDP_IF_J2.13
- net HADRCLK*: now also 4421_PDP_IF_J2.68
- net BUSA10*: now reaches 4421_PDP_IF_J2.15
- net BUSA10*: now also UNIBUS_XFER_J1.21 (Pin_21)
- net BUSA09*: now reaches 4421_PDP_IF_J2.17
- net BUSA09*: now also UNIBUS_XFER_J1.19 (Pin_19)
- net DMAIND: now reaches 4421_PDP_IF_J2.18
- net BUSD11*: now reaches 4421_PDP_IF_J2.19
- net BUSD11*: now also UNIBUS_XFER_J1.24 (Pin_24)
- net RUNIND: now reaches 4421_PDP_IF_J2.20
- net BUSD10*: now reaches 4421_PDP_IF_J2.21
- net BUSD10*: now also UNIBUS_XFER_J1.22 (Pin_22)
- net BUSNPGOUT: now reaches 4421_PDP_IF_J2.22
- net BUSNPGOUT: now also UNIBUS_XFER_J1.48 (Pin_48)
- net BUSD09*: now reaches 4421_PDP_IF_J2.25
- net BUSD09*: now also UNIBUS_XFER_J1.20 (Pin_20)
- net BUSD08*: now reaches 4421_PDP_IF_J2.27
- net BUSD08*: now also UNIBUS_XFER_J1.18 (Pin_18)
- net BUSD07*: now reaches 4421_PDP_IF_J2.29
- net BUSD07*: now also UNIBUS_XFER_J1.16 (Pin_16)
- net BUSD06*: now reaches 4421_PDP_IF_J2.31
- net BUSD06*: now also UNIBUS_XFER_J1.14 (Pin_14)
- net BUSSACK*: now reaches 4421_PDP_IF_J2.32
- net BUSSACK*: now also UNIBUS_XFER_J1.40 (Pin_40)
- net BUSNPR*: now reaches 4421_PDP_IF_J2.34
- net BUSNPR*: now also UNIBUS_XFER_J1.42 (Pin_42)
- net BUSD05*: now reaches 4421_PDP_IF_J2.35
- net BUSD05*: now also UNIBUS_XFER_J1.12 (Pin_12)
- net BUSD04*: now reaches 4421_PDP_IF_J2.37
- net BUSD04*: now also UNIBUS_XFER_J1.10 (Pin_10)
- net BUSA08*: now reaches 4421_PDP_IF_J2.47
- net BUSA08*: now also UNIBUS_XFER_J1.17 (Pin_17)
- net BUSSSYN*: now reaches 4421_PDP_IF_J2.48
- net BUSSSYN*: now also UNIBUS_XFER_J1.46 (Pin_46)
- net BUSA07*: now reaches 4421_PDP_IF_J2.49
- net BUSA07*: now also UNIBUS_XFER_J1.15 (Pin_15)
- net BUSINTR*: now reaches 4421_PDP_IF_J2.5
- net BUSINTR*: now also UNIBUS_XFER_J1.39 (Pin_39)
- net BUSC01*: now reaches 4421_PDP_IF_J2.50
- net BUSC01*: now also UNIBUS_XFER_J1.38 (Pin_38)
- net !HRSET: now reaches 4421_PDP_IF_J2.52
- net BUSA06*: now reaches 4421_PDP_IF_J2.53
- net BUSA06*: now also UNIBUS_XFER_J1.13 (Pin_13)
- net BUSINIT*: now reaches 4421_PDP_IF_J2.54
- net BUSINIT*: now also UNIBUS_XFER_J1.44 (Pin_44)
- net BUSA05*: now reaches 4421_PDP_IF_J2.55
- net BUSA05*: now also UNIBUS_XFER_J1.11 (Pin_11)
- net BUSMSYN*: now reaches 4421_PDP_IF_J2.56
- net BUSMSYN*: now also UNIBUS_XFER_J1.43 (Pin_43)
- net BUSD03*: now reaches 4421_PDP_IF_J2.57
- net BUSD03*: now also UNIBUS_XFER_J1.8 (Pin_8)
- net BUSD02*: now reaches 4421_PDP_IF_J2.59
- net BUSD02*: now also UNIBUS_XFER_J1.6 (Pin_6)
- net BUSBGOUT: now reaches 4421_PDP_IF_J2.6
- net BUSBGOUT: now also UNIBUS_XFER_J1.50 (Pin_50)
- net BUSD01*: now reaches 4421_PDP_IF_J2.63
- net BUSD01*: now also UNIBUS_XFER_J1.4 (Pin_4)
- net BUSD00*: now reaches 4421_PDP_IF_J2.65
- net BUSD00*: now also UNIBUS_XFER_J1.2 (Pin_2)
- net PWFAIL*: now reaches 4421_PDP_IF_J2.66
- net BUSBR*: now reaches 4421_PDP_IF_J2.7
- net BUSBR*: now also UNIBUS_XFER_J1.41 (Pin_41)
- net HADR2HD*: now reaches 4421_PDP_IF_J2.70
- net HADR2HD*: now also 4421_PDP_IF_J2.91
- net INT06*: now reaches 4421_PDP_IF_J2.76
- net INT07*: now reaches 4421_PDP_IF_J2.78
- net BUSA04*: now reaches 4421_PDP_IF_J2.87
- net BUSA04*: now also UNIBUS_XFER_J1.9 (Pin_9)
- net BUSA03*: now reaches 4421_PDP_IF_J2.89
- net BUSA03*: now also UNIBUS_XFER_J1.7 (Pin_7)
- net BUSA12*: now reaches 4421_PDP_IF_J2.9
- net BUSA12*: now also UNIBUS_XFER_J1.25 (Pin_25)
- net BUSA02*: now reaches 4421_PDP_IF_J2.93
- net BUSA02*: now also UNIBUS_XFER_J1.5 (Pin_5)
- net BUSA01*: now reaches 4421_PDP_IF_J2.95
- net BUSA01*: now also UNIBUS_XFER_J1.3 (Pin_3)
Other:
- note added: "UNIBUS XFER"

Commit message: 2026/1/6
Parts:
- removed Spare2_J1, Spare2_J2: Conn_02x50_100pin, symbol User:Conn_02x50_100pin
- 4401_FA_J1, 4401_FA_J2, 4402_DPL_J1, 4402_DPL_J2, 4402_DPR_J1, 4402_DPR_J2, 4408_P3_J1, 4408_P3_J2, 4422_P1_J3, 4422_P1_J4, 4423_P2_J1, 4423_P2_J2, 4424_MD_J1, 4424_MD_J2, 4425_TM_J1, 4425_TM_J2, 4426_FM_J1, 4426_FM_J2, Spare1_J1, Spare1_J2: footprint (none) -> User:120pin_Edge_Connector
- 4421_PDP_IF_J1, 4421_PDP_IF_J2, 4429_FMT_J1, 4429_FMT_J2, Spare2_J3, Spare2_J4: footprint (none) -> User:100pin_Edge_Connector
- UNIBUS_XFER_J1: footprint (none) -> Connector_PinHeader_2.54mm:PinHeader_2x25_P2.54mm_Vertical
Other:
- moved on the sheet: 4421_PDP_IF_J1, 4421_PDP_IF_J2, 4429_FMT_J1, 4429_FMT_J2, Spare2_J3, Spare2_J4, UNIBUS_XFER_J1
