File: FPS 100/Backplane/Backplane.kicad_pcb (KiCad board)
At the start: 6 copper layers, 27 parts

Commit message: 2026/1/7
Connections:
- 4401_FA_J1 pad 30: FAUNFL* -> FAUNF*
- 4401_FA_J1 pad 32: FAOVFL* -> FAOVF*
- 4401_FA_J1 pad 33: SCN -> SCIN
- 4401_FA_J1 pad 35: unconnected-(4401_FA_J1-Pad35) -> DE07*
- 4401_FA_J1 pad 37: DE07* -> unconnected-(4401_FA_J1-Pad37)
- 4401_FA_J2 pad 100: unconnected-(4401_FA_J2-Pad100) -> FRCINH*
- 4422_P1_J3 pad 16: FAZERO* -> FAZRO*
Routing:
- net DPMBS21*: track 0.00 -> 421.1 mm, vias 0 -> 8
- net DPMBS20*: track 0.00 -> 409.5 mm, vias 0 -> 13
- net MDCR3*: track 0.00 -> 356.1 mm, vias 0 -> 3
- net MIA*: track 0.00 -> 326.3 mm, vias 0 -> 2
- net MIB*: track 0.00 -> 322.4 mm, vias 0 -> 2
- net DPMBS22*: track 0.00 -> 304.8 mm, vias 0 -> 10
- net MALD*: track 0.00 -> 291.4 mm, vias 0 -> 2
- net MACE*: track 0.00 -> 275.5 mm, vias 0 -> 2
- net SETATMA*: track 0.00 -> 244.1 mm, vias 0 -> 2
- net DPMBS23*: track 0.00 -> 213.4 mm, vias 0 -> 5
- net PS24*A: track 0.00 -> 208.5 mm, vias 0 -> 2
- net MDI39: track 0.00 -> 208.5 mm, vias 0 -> 4
- net MDI38: track 0.00 -> 208.0 mm, vias 0 -> 6
- net PS25*A: track 0.00 -> 201.4 mm, vias 0 -> 2
- net PSA15*: track 0.00 -> 151.8 mm, vias 0 -> 2
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
Commit message: 2026/1/7
Parts:
- moved UNIBUS_XFER_J1 46.8 mm to (350.1, 414.4)
Connections:
- 4402_DPL_J2 pad 56: DPMBS24* -> DPMBS23*
- 4408_P3_J1 pad 25: IHRSET* -> !HRSET*
- 4408_P3_J1 pad 9: !WRTR -> !WRTR*
- 4421_PDP_IF_J1 pad 42: B2ID -> B2IO
- 4421_PDP_IF_J1 pad 52: unconnected-(4421_PDP_IF_J1-Pad52) -> !HRSET*
- 4422_P1_J3 pad 101: 375LD* -> 376LD*
Routing:
- net FADD*: track 0.00 -> 392.1 mm, vias 0 -> 3
- net CB14*: track 0.00 -> 361.5 mm, vias 0 -> 2
- net CB15*: track 0.00 -> 357.3 mm, vias 0 -> 3
- net CB17*: track 0.00 -> 356.5 mm, vias 0 -> 3
- net CB19*: track 0.00 -> 354.3 mm, vias 0 -> 3
- net CB16*: track 0.00 -> 352.2 mm, vias 0 -> 2
- net CB18*: track 0.00 -> 349.9 mm, vias 0 -> 2
- net LDSR*: track 0.00 -> 333.0 mm, vias 0 -> 1
- net I+H14: track 0.00 -> 315.8 mm, vias 0 -> 1
- net I+H13: track 0.00 -> 296.3 mm, vias 0 -> 2
- net REFSYNC*: track 0.00 -> 291.3 mm, vias 0 -> 4
- net DMA13*: track 0.00 -> 289.7 mm, vias 0 -> 1
- net DMA15*: track 0.00 -> 289.3 mm, vias 0 -> 1
- net DMA12*: track 0.00 -> 287.2 mm, vias 0 -> 1
- net DMA14*: track 0.00 -> 286.7 mm, vias 0 -> 1
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Other:
- board outline added: 379.6 x 225.7 mm

Commit message: 2026/1/7
Routing:
- net MD02*: track 0.00 -> 409.6 mm, vias 0 -> 4
- net MD03*: track 0.00 -> 409.0 mm, vias 0 -> 4
- net DPEBS03*: track 0.00 -> 285.4 mm, vias 0 -> 6
- net PNL08*: track 0.00 -> 250.9 mm, vias 0 -> 5
- net PNL09*: track 0.00 -> 225.3 mm, vias 0 -> 4
- net PNL11*: track 0.00 -> 224.5 mm, vias 0 -> 4
- net PNL10*: track 0.00 -> 221.3 mm, vias 0 -> 4
- net DA11*: track 0.00 -> 211.0 mm, vias 0 -> 3
- net DA10*: track 0.00 -> 199.3 mm, vias 0 -> 3
- net B2IO: track 50.4 -> 51.0 mm

Commit message: 2026/1/8
Connections:
- 4421_PDP_IF_J1 pad 52: !HRSET* -> unconnected-(4421_PDP_IF_J1-Pad52)
- 4421_PDP_IF_J2 pad 52: !HRSET -> !HRSET*
Routing:
- net +5V: track 1476.8 -> 2785.5 mm, vias 0 -> 2
- net FAM02*: track 0.00 -> 233.5 mm, vias 0 -> 5
- net FAE08*: track 0.00 -> 228.7 mm, vias 0 -> 3
- net FAM01*: track 0.00 -> 228.6 mm, vias 0 -> 3
- net FAM03*: track 0.00 -> 225.1 mm, vias 0 -> 2
- net FAM00*: track 0.00 -> 223.2 mm, vias 0 -> 2
- net FMM03*: track 0.00 -> 217.5 mm, vias 0 -> 4
- net FMM02*: track 0.00 -> 215.2 mm, vias 0 -> 4
- net FMM00*: track 0.00 -> 214.3 mm, vias 0 -> 3
- net FMM01*: track 0.00 -> 213.9 mm, vias 0 -> 3
- net FAE11*: track 0.00 -> 194.3 mm, vias 0 -> 2
- net FAE10*: track 0.00 -> 192.8 mm, vias 0 -> 2
- net FAE09*: track 0.00 -> 192.3 mm, vias 0 -> 2
- net A1MBS01*: track 0.00 -> 175.4 mm, vias 0 -> 2
- net A1MBS00*: track 0.00 -> 174.9 mm, vias 0 -> 2
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Other:
- board size 379.6 x 225.7 mm -> 384.7 x 240.4 mm

Commit message: 2026/1/8
Connections:
- 4408_P3_J1 pad 116: NCP* -> NOP*
- 4408_P3_J1 pad 12: !M1CLK -> !MICLK
- 4408_P3_J2 pad 113: INTCP -> INTOP
Routing:
- net DP2M2: track 0.00 -> 244.0 mm, vias 0 -> 1
- net A1MBS06*: track 0.00 -> 184.3 mm, vias 0 -> 2
- net A2MBS01*: track 0.00 -> 180.4 mm, vias 0 -> 3
- net FMM05*: track 0.00 -> 178.2 mm, vias 0 -> 3
- net A2MBS00*: track 0.00 -> 177.3 mm, vias 0 -> 3
- net A1MBS07*: track 0.00 -> 175.8 mm, vias 0 -> 2
- net FMM04*: track 0.00 -> 172.8 mm, vias 0 -> 3
- net FAM04*: track 0.00 -> 168.8 mm, vias 0 -> 3
- net FAM05*: track 0.00 -> 166.6 mm, vias 0 -> 2
- net FMM07*: track 0.00 -> 166.2 mm, vias 0 -> 3
- net FMM06*: track 0.00 -> 162.2 mm, vias 0 -> 2
- net DP2DP: track 0.00 -> 143.2 mm, vias 0 -> 4
- net FMM15*: track 0.00 -> 118.6 mm, vias 0 -> 2
- net A1MBS04*: track 0.00 -> 117.3 mm, vias 0 -> 2
- net A1MBS13*: track 0.00 -> 116.7 mm, vias 0 -> 2
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
Commit message: 2026/1/8
Connections:
- 4421_PDP_IF_J1 pad 64: DAM01* -> DMA01*
- 4423_P2_J1 pad 39: PLN00* -> PNL00*
- 4423_P2_J1 pad 40: PLN01* -> PNL01*
- 4423_P2_J1 pad 41: PLN02* -> PNL02*
- 4423_P2_J1 pad 42: PLN03* -> PNL03*
- 4423_P2_J1 pad 43: PLN04* -> PNL04*
- 4423_P2_J1 pad 44: PLN05* -> PNL05*
- 4423_P2_J1 pad 45: PLN06* -> PNL06*
- 4423_P2_J1 pad 46: PLN07* -> PNL07*
- 4423_P2_J1 pad 63: PLN08* -> PNL08*
- 4423_P2_J1 pad 64: PLN09* -> PNL09*
- 4423_P2_J1 pad 65: PLN10* -> PNL10*
- 4423_P2_J1 pad 66: PLN11* -> PNL11*
- 4423_P2_J1 pad 67: PLN12* -> PNL12*
- 4423_P2_J1 pad 68: PLN13* -> PNL13*
- 4423_P2_J1 pad 69: PLN14* -> PNL14*
- 4423_P2_J1 pad 70: PLN15* -> PNL15*
- 4425_TM_J1 pad 102: MIEBS10* -> M1EBS10*
- 4425_TM_J1 pad 104: MIEBS11* -> M1EBS11*
- 4425_TM_J1 pad 106: MIMBS00* -> M1MBS00*
- 4425_TM_J1 pad 108: MIMBS01* -> M1MBS01*
- 4425_TM_J1 pad 110: MIMBS02* -> M1MBS02*
- 4425_TM_J1 pad 112: MIMBS03* -> M1MBS03*
- 4425_TM_J1 pad 114: MIMBS04* -> M1MBS04*
- 4425_TM_J1 pad 116: MIMBS05* -> M1MBS05*
- 4425_TM_J1 pad 72: MIEBS02* -> M1EBS02*
- 4425_TM_J1 pad 74: MIEBS03* -> M1EBS03*
- 4425_TM_J1 pad 76: MIEBS04* -> M1EBS04*
- 4425_TM_J1 pad 78: MIEBS05* -> M1EBS05*
- 4425_TM_J1 pad 80: MIEBS06* -> M1EBS06*
- 4425_TM_J1 pad 82: MIEBS07* -> M1EBS07*
- 4425_TM_J1 pad 84: MIEBS08* -> M1EBS08*
- 4425_TM_J1 pad 86: MIEBS09* -> M1EBS09*
- 4425_TM_J2 pad 100: MIMBS23* -> M1MBS23*
- 4425_TM_J2 pad 102: MIMBS24* -> M1MBS24*
- 4425_TM_J2 pad 104: MIMBS25* -> M1MBS25*
- 4425_TM_J2 pad 106: MIMBS26* -> M1MBS26*
- 4425_TM_J2 pad 108: MIMBS27* -> M1MBS27*
- 4425_TM_J2 pad 22: MIMBS06* -> M1MBS06*
- 4425_TM_J2 pad 24: MIMBS07* -> M1MBS07*
- 4425_TM_J2 pad 26: MIMBS08* -> M1MBS08*
- 4425_TM_J2 pad 28: MIMBS09* -> M1MBS09*
- 4425_TM_J2 pad 30: MIMBS10* -> M1MBS10*
- 4425_TM_J2 pad 32: MIMBS11* -> M1MBS11*
- 4425_TM_J2 pad 34: MIMBS12* -> M1MBS12*
- 4425_TM_J2 pad 36: MIMBS13* -> M1MBS13*
- 4425_TM_J2 pad 56: MIMBS14* -> M1MBS14*
- 4425_TM_J2 pad 58: MIMBS15* -> M1MBS15*
- 4425_TM_J2 pad 60: MIMBS16* -> M1MBS16*
- 4425_TM_J2 pad 62: MIMBS17* -> M1MBS17*
- 4425_TM_J2 pad 64: MIMBS18* -> M1MBS18*
- 4425_TM_J2 pad 66: MIMBS19* -> M1MBS19*
- 4425_TM_J2 pad 68: MIMBS20* -> M1MBS20*
- 4425_TM_J2 pad 70: MIMBS21* -> M1MBS21*
- 4425_TM_J2 pad 98: MIMBS22* -> M1MBS22*
Routing:
- net MDI02: track 0.00 -> 352.2 mm, vias 0 -> 2
- net MDI05: track 0.00 -> 350.7 mm, vias 0 -> 3
- net MDI03: track 0.00 -> 348.0 mm, vias 0 -> 2
- net INTR*: track 0.00 -> 229.3 mm, vias 0 -> 1
- net DP2A2M: track 0.00 -> 17.8 mm, vias 0 -> 2
- net Y2A2: track 0.00 -> 16.8 mm
- net YLMCLKE*: track 0.00 -> 16.2 mm, vias 0 -> 2
- net DP2A1: track 0.00 -> 16.2 mm, vias 0 -> 2
- net XLMCLKE*: track 0.00 -> 16.0 mm, vias 0 -> 2
- net Y2M1: track 0.00 -> 15.9 mm, vias 0 -> 2
- net Y2M2: track 0.00 -> 15.8 mm, vias 0 -> 2
- net DP2M1: track 0.00 -> 15.3 mm, vias 0 -> 2
- net Y2DP: track 0.00 -> 15.2 mm, vias 0 -> 2
- net Y2A1: track 0.00 -> 15.2 mm, vias 0 -> 2
- net A1EBS02*: track 48.3 -> 48.9 mm

Commit message: 2026/1/9
Routing:
- net MD00*: track 0.00 -> 163.7 mm, vias 0 -> 3
- net FAM22*: track 0.00 -> 138.1 mm, vias 0 -> 6
- net FAM21*: track 0.00 -> 137.5 mm, vias 0 -> 2
- net FAM20*: track 0.00 -> 135.4 mm, vias 0 -> 2
- net FMM14*: track 0.00 -> 125.5 mm, vias 0 -> 3
- net A1EBS02*: track 48.9 -> 170.1 mm, vias 2 -> 6
- net FMM12*: track 0.00 -> 119.3 mm, vias 0 -> 2
- net FMM13*: track 0.00 -> 103.5 mm, vias 0 -> 2
- net A2MBS11*: track 0.00 -> 61.2 mm, vias 0 -> 1
- net A2MBS10*: track 0.00 -> 59.9 mm, vias 0 -> 1
- net A2MBS09*: track 0.00 -> 59.3 mm, vias 0 -> 1
- net A2MBS08*: track 0.00 -> 57.6 mm, vias 0 -> 1
- net MD02*: track 409.6 -> 408.6 mm
